File: Infra-pHAT.kicad_pcb (KiCad board)
At the start: 2 copper layers, 65 x 30 mm, 25 parts, among them Q1 BC817, U1 CAT24C32WI-GT3

Commit message: Update logo, texts and IRTX position
Signed-off-by: Leon Anavi <leon@anavi.org>
Parts:
- moved IRRX 4.08 mm to (166.8, 99.7)
- moved R4 0.20 mm to (159.6, 91.6)
- moved ? 0.10 mm to (175.2, 101.7)
- renumbered IRRX1 to IRRX
Routing:
- net Net-(C2-Pad1): track 11.4 -> 9.96 mm
- net Net-(IRRX1-Pad1): track 43.7 -> 45.1 mm
Changed lines of the file:
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@@
     (area 136.817429 66.3 225.182572 110.000001)
     (thickness 1.6)
-    (drawings 22)
-    (tracks 236)
+    (drawings 21)
+    (tracks 239)
     (zones 0)
     (modules 25)
@@
     (visible_elements FFFEFFFF)
     (pcbplotparams
-      (layerselection 0x010f0_80000001)
+      (layerselection 0x010e0_80000001)
       (usegerberextensions true)
       (excludeedgelayer true)
@@
     (tags "capacitor 0805")
     (attr smd)
-    (fp_text reference C2 (at 3.71 -0.11 180) (layer F.SilkS)
+    (fp_text reference C2 (at 0.06 2.04 180) (layer F.SilkS)
       (effects (font (size 1 1) (thickness 0.15)))
     )
@@
     (tags SOT-23)
     (attr smd)
-    (fp_text reference Q1 (at -2.75 -1.15 180) (layer F.SilkS)
+    (fp_text reference Q1 (at 0 -2.6 180) (layer F.SilkS)
       (effects (font (size 1 1) (thickness 0.15)))
     )
@@
     (tags "resistor 0603")
     (attr smd)
-    (fp_text reference R2 (at 0 -1.9 180) (layer F.SilkS)
+    (fp_text reference R2 (at 0 -1.7 180) (layer F.SilkS)
       (effects (font (size 1 1) (thickness 0.15)))
     )
@@
   )
   (module Resistors_SMD:R_0603_HandSoldering (layer F.Cu)
-    (at 159.4 91.6)
+    (at 159.6 91.6)
     (descr "Resistor SMD 0603, hand soldering")
     (tags "resistor 0603")
     (attr smd)
-    (fp_text reference R4 (at 3.2 0.05) (layer F.SilkS)
+    (fp_text reference R4 (at 0.1 1.8) (layer F.SilkS)
       (effects (font (size 1 1) (thickness 0.15)))
     )
@@
   )
   (module myfootprint:TSOP38X (layer F.Cu)
-    (at 162.726 99.561)
-    (fp_text reference IRRX1 (at 0.074 0.339) (layer F.SilkS)
+    (at 166.8 99.7)
+    (fp_text reference IRRX (at 0.074 0.339) (layer F.SilkS)
       (effects (font (size 1 1) (thickness 0.15)))
     )
@@
   )
   (module logo:anavi-logo (layer F.Cu)
-    (at 175.3 101.7)
+    (at 175.2 101.7)
     (fp_text reference "" (at 0 0) (layer F.SilkS) hide
       (effects (font (thickness 0.3)))
@@
       (effects (font (thickness 0.3)))
     )
-    (fp_poly (pts (xy 1.693334 1.693334) (xy -1.693333 1.693334) (xy -1.693333 -1.439333) (xy -1.27 -1.439333)
-      (xy -1.27 1.27) (xy 1.439334 1.27) (xy 1.439334 -1.439333) (xy -1.27 -1.439333)
-      (xy -1.693333 -1.439333) (xy -1.693333 -1.778) (xy 1.693334 -1.778) (xy 1.693334 1.693334)) (layer F.SilkS) (width 0.01))
+    (fp_poly (pts (xy 1.693334 1.693334) (xy -1.693333 1.693334) (xy -1.693333 -1.524) (xy -1.185333 -1.524)
+      (xy -1.185333 1.185334) (xy 1.439334 1.185334) (xy 1.439334 -1.524) (xy -1.185333 -1.524)
+      (xy -1.693333 -1.524) (xy -1.693333 -1.778) (xy 1.693334 -1.778) (xy 1.693334 1.693334)) (layer F.SilkS) (width 0.01))
   )
   (gr_text "Rev 1.0 (c) 2017" (at 182.8 102) (layer F.SilkS)
@@
     (arrow2b (pts (xy 210 69) (xy 211.126504 68.413579)))
   )
-  (gr_line (start 152 78.5) (end 155.1 78.5) (angle 90) (layer F.Mask) (width 0.2))
   (gr_line (start 152 78.46) (end 152 77.46) (angle 90) (layer B.SilkS) (width 0.2))
   (gr_line (start 148.5011 102.0036) (end 148.5011 78.0036) (layer Edge.Cuts) (width 0.1))
@@
   (segment (start 197.25 100.5) (end 197.27 100.45) (width 0.5) (layer F.Cu) (net 2) (status 80000))
   (segment (start 169.31 96.64) (end 169.291 96.647) (width 0.5) (layer F.Cu) (net 3) (status 80000))
-  (segment (start 169.291 96.647) (end 165.227 100.711) (width 0.5) (layer F.Cu) (net 3) (status 80000))
-  (segment (start 165.227 100.711) (end 165.227 102.108) (width 0.5) (layer F.Cu) (net 3) (status 80000))
-  (segment (start 165.227 102.108) (end 165.266 102.101) (width 0.5) (layer F.Cu) (net 3) (status 80000))
+  (segment (start 169.291 96.647) (end 169.291 102.235) (width 0.5) (layer F.Cu) (net 3) (status 80000))
+  (segment (start 169.291 102.235) (end 169.34 102.24) (width 0.5) (layer F.Cu) (net 3) (status 80000))
+  (segment (start 169.31 96.64) (end 169.291 96.647) (width 0.5) (layer F.Cu) (net 3) (status 80000))
+  (segment (start 169.301 102.247) (end 169.34 102.24) (width 0.5) (layer F.Cu) (net 3) (status 80030))
   (segment (start 169.31 96.64) (end 169.25 96.75) (width 0.5) (layer F.Cu) (net 3) (status 80000))
   (segment (start 169.25 96.75) (end 169.25 92.75) (width 0.5) (layer F.Cu) (net 3) (status 80000))
@@
   (segment (start 210 94) (end 209.97 94.1) (width 0.5) (layer B.Cu) (net 6) (status 80000))
   (segment (start 160.65 85.59924) (end 160.655 85.598) (width 0.5) (layer F.Cu) (net 7) (status 80000))
+  (segment (start 160.655 85.598) (end 160.655 91.567) (width 0.5) (layer F.Cu) (net 7) (status 80000))
+  (segment (start 160.655 91.567) (end 160.7 91.6) (width 0.5) (layer F.Cu) (net 7) (status 80000))
+  (segment (start 160.65 85.59924) (end 160.655 85.598) (width 0.5) (layer F.Cu) (net 7) (status 80000))
   (segment (start 160.655 85.598) (end 161.417 85.598) (width 0.5) (layer F.Cu) (net 7) (status 80000))
   (segment (start 161.417 85.598) (end 162.306 86.487) (width 0.5) (layer F.Cu) (net 7) (status 80000))
@@
   (segment (start 169.545 79.756) (end 169.55 79.8) (width 0.5) (layer F.Cu) (net 7) (status 80000))
   (segment (start 160.65 85.59924) (end 160.655 85.598) (width 0.5) (layer F.Cu) (net 7) (status 80000))
-  (segment (start 160.655 85.598) (end 160.655 88.519) (width 0.5) (layer F.Cu) (net 7) (status 80000))
-  (segment (start 160.655 88.519) (end 160.528 88.646) (width 0.5) (layer F.Cu) (net 7) (status 80000))
-  (segment (start 160.528 88.646) (end 160.528 91.567) (width 0.5) (layer F.Cu) (net 7) (status 80000))
-  (segment (start 160.528 91.567) (end 160.5 91.6) (width 0.5) (layer F.Cu) (net 7) (status 80000))
+  (segment (start 160.728 91.567) (end 160.7 91.6) (width 0.5) (layer F.Cu) (net 7) (status 80030))
   (segment (start 189.87 77.26) (end 189.865 77.216) (width 0.5) (layer B.Cu) (net 8) (status 80000))
   (segment (start 189.865 77.216) (end 191.008 76.073) (width 0.5) (layer B.Cu) (net 8) (status 80000))
@@
   (segment (start 168.3 82.05) (end 172.18 85.93) (width 0.254) (layer F.Cu) (net 13))
   (segment (start 172.18 85.93) (end 172.18 86.5) (width 0.254) (layer F.Cu) (net 13))
-  (segment (start 169.5 77.25) (end 168.5 76.25) (width 0.5) (layer B.Cu) (net 14) (status 80000))
-  (segment (start 160.25 86.25) (end 160.25 102) (width 0.5) (layer B.Cu) (net 14) (status 80000))
-  (segment (start 155.25 81.25) (end 160.25 86.25) (width 0.5) (layer B.Cu) (net 14) (status 80000))
-  (segment (start 155.25 75.75) (end 155.25 81.25) (width 0.5) (layer B.Cu) (net 14) (status 80000))
-  (segment (start 168.5 75.75) (end 155.25 75.75) (width 0.5) (layer B.Cu) (net 14) (status 80000))
-  (segment (start 168.5 76.25) (end 168.5 75.75) (width 0.5) (layer B.Cu) (net 14) (status 80000))
+  (segment (start 169.55 77.26) (end 169.545 77.216) (width 0.5) (layer B.Cu) (net 14) (status 80000))
+  (segment (start 169.545 77.216) (end 168.402 76.073) (width 0.5) (layer B.Cu) (net 14) (status 80000))
+  (segment (start 168.402 76.073) (end 168.402 75.819) (width 0.5) (layer B.Cu) (net 14) (status 80000))
+  (segment (start 168.402 75.819) (end 155.448 75.819) (width 0.5) (layer B.Cu) (net 14) (status 80000))
+  (segment (start 155.448 75.819) (end 155.448 81.28) (width 0.5) (layer B.Cu) (net 14) (status 80000))
+  (segment (start 155.448 81.28) (end 164.211 90.043) (width 0.5) (layer B.Cu) (net 14) (status 80000))
+  (segment (start 164.211 90.043) (end 164.211 102.235) (width 0.5) (layer B.Cu) (net 14) (status 80000))
+  (segment (start 164.211 102.235) (end 164.26 102.24) (width 0.5) (layer B.Cu) (net 14) (status 80000))
   (segment (start 169.55 77.26) (end 169.5 77.25) (width 0.5) (layer B.Cu) (net 14) (status 80000))
-  (segment (start 160.25 102) (end 160.186 102.101) (width 0.5) (layer B.Cu) (net 14) (status 80000))
+  (segment (start 164.324 102.139) (end 164.26 102.24) (width 0.5) (layer B.Cu) (net 14) (status 80030))
   (segment (start 159.7 87.59822) (end 159.639 87.63) (width 0.5) (layer F.Cu) (net 15) (status 80000))
   (segment (start 159.639 87.63) (end 159.512 87.757) (width 0.5) (layer F.Cu) (net 15) (status 80000))

Commit message: Update name
Signed-off-by: Leon Anavi <leon@anavi.org>
Other:
- board text added: "ANAVI Infrared pHAT"
- board text removed: "ANAVI Infra pHAT"
Changed lines of the file:
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@@
     (effects (font (size 0.8 0.8) (thickness 0.15)))
   )
-  (gr_text "ANAVI Infra pHAT" (at 183.9 100.4) (layer F.SilkS)
+  (gr_text "ANAVI Infrared pHAT" (at 185.1 100.5) (layer F.SilkS)
     (effects (font (size 1 1) (thickness 0.25)))
   )

Commit message: Infra-pHAT.kicad_pcb: Add assembly instructions
Signed-off-by: Leon Anavi <leon@anavi.org>
Other:
- board text added: "100nF"
- board text added: "10K"
- board text added: "1K"
- board text added: "4,7K"
- board text added: "4,7pF"
- board text added: "470"
- board text added: "BC817"
Changed lines of the file:
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@@
     (area 136.817429 66.3 225.182572 110.000001)
     (thickness 1.6)
-    (drawings 21)
+    (drawings 31)
     (tracks 239)
     (zones 0)
@@
   )
   (layers
-    (0 F.Cu signal)
-    (31 B.Cu signal)
-    (32 B.Adhes user)
-    (33 F.Adhes user)
-    (34 B.Paste user)
-    (35 F.Paste user)
+    (0 F.Cu signal hide)
+    (31 B.Cu signal hide)
+    (32 B.Adhes user hide)
+    (33 F.Adhes user hide)
+    (34 B.Paste user hide)
+    (35 F.Paste user hide)
     (36 B.SilkS user hide)
-    (37 F.SilkS user)
-    (38 B.Mask user)
-    (39 F.Mask user)
-    (40 Dwgs.User user)
-    (41 Cmts.User user)
+    (37 F.SilkS user hide)
+    (38 B.Mask user hide)
+    (39 F.Mask user hide)
+    (40 Dwgs.User user hide)
+    (41 Cmts.User user hide)
     (42 Eco1.User user hide)
     (43 Eco2.User user hide)
     (44 Edge.Cuts user)
-    (45 Margin user)
-    (46 B.CrtYd user)
+    (45 Margin user hide)
+    (46 B.CrtYd user hide)
     (47 F.CrtYd user)
     (48 B.Fab user hide)
-    (49 F.Fab user hide)
+    (49 F.Fab user)
   )
   (setup
@@
     (pad_to_mask_clearance 0)
     (aux_axis_origin 0 0)
-    (visible_elements FFFEFFFF)
+    (visible_elements FFFFF97F)
     (pcbplotparams
       (layerselection 0x010e0_80000001)
@@
       (drillshape 0)
       (scaleselection 1)
-      (outputdirectory plots/rev-1.0/))
+      (outputdirectory schemes/))
   )
   (net 0 "")
@@
       (effects (font (size 1 1) (thickness 0.15)))
     )
-    (fp_text value 0.1 (at 0 1.9 90) (layer F.Fab)
+    (fp_text value 0.1 (at 0 1.9 90) (layer F.Fab) hide
       (effects (font (size 1 1) (thickness 0.15)))
     )
@@
       (effects (font (size 1 1) (thickness 0.15)))
     )
-    (fp_text value 4.7 (at 0 2.1 180) (layer F.Fab)
+    (fp_text value 4.7 (at 0 2.1 180) (layer F.Fab) hide
       (effects (font (size 1 1) (thickness 0.15)))
     )
@@
       (effects (font (size 1 1) (thickness 0.15)))
     )
-    (fp_text value L-53F3BT (at 1.524 -3.937 90) (layer F.Fab)
+    (fp_text value L-53F3BT (at 1.524 -3.937 90) (layer F.Fab) hide
       (effects (font (size 1 1) (thickness 0.15)))
     )
@@
       (effects (font (size 1 1) (thickness 0.15)))
     )
-    (fp_text value L-53F3BT (at 1.524 -3.937 90) (layer F.Fab)
+    (fp_text value L-53F3BT (at 1.524 -3.937 90) (layer F.Fab) hide
       (effects (font (size 1 1) (thickness 0.15)))
     )
@@
       (effects (font (size 1 1) (thickness 0.15)))
     )
-    (fp_text value JUMPER (at 0 -3.1) (layer F.Fab)
+    (fp_text value JUMPER (at 0 -3.1) (layer F.Fab) hide
       (effects (font (size 1 1) (thickness 0.15)))
     )
@@
       (effects (font (size 1 1) (thickness 0.15)))
     )
-    (fp_text value BC817 (at 0 2.3 180) (layer F.Fab)
+    (fp_text value BC817 (at 0 2.3 180) (layer F.Fab) hide
       (effects (font (size 1 1) (thickness 0.15)))
     )
@@
       (effects (font (size 1 1) (thickness 0.15)))
     )
-    (fp_text value 1K (at 0 1.9 270) (layer F.Fab)
+    (fp_text value 1K (at 0 1.9 270) (layer F.Fab) hide
       (effects (font (size 1 1) (thickness 0.15)))
     )
@@
       (effects (font (size 1 1) (thickness 0.15)))
     )
-    (fp_text value 4.7K (at 0 1.9 180) (layer F.Fab)
+    (fp_text value 4.7K (at 0 1.9 180) (layer F.Fab) hide
       (effects (font (size 1 1) (thickness 0.15)))
     )
@@
       (effects (font (size 1 1) (thickness 0.15)))
     )
-    (fp_text value 4.7K (at 0 1.9 180) (layer F.Fab)
+    (fp_text value 4.7K (at 0 1.9 180) (layer F.Fab) hide
       (effects (font (size 1 1) (thickness 0.15)))
     )
@@
       (effects (font (size 1 1) (thickness 0.15)))
     )
-    (fp_text value 10K (at 0 1.9) (layer F.Fab)
+    (fp_text value 10K (at 0 1.9) (layer F.Fab) hide
       (effects (font (size 1 1) (thickness 0.15)))
     )
@@
       (effects (font (size 1 1) (thickness 0.15)))
     )
-    (fp_text value 470 (at 0 1.9 270) (layer F.Fab)
+    (fp_text value 470 (at 0 1.9 270) (layer F.Fab) hide
       (effects (font (size 1 1) (thickness 0.15)))
     )
@@
       (effects (font (size 1 1) (thickness 0.15)))
     )
-    (fp_text value 4.7K (at 0 1.9 270) (layer F.Fab)
+    (fp_text value 4.7K (at 0 1.9 270) (layer F.Fab) hide
       (effects (font (size 1 1) (thickness 0.15)))
     )
@@
       (effects (font (size 1 1) (thickness 0.15)))
     )
-    (fp_text value 4.7K (at 0 1.9 270) (layer F.Fab)
+    (fp_text value 4.7K (at 0 1.9 270) (layer F.Fab) hide
       (effects (font (size 1 1) (thickness 0.15)))
     )
@@
       (effects (font (size 1 1) (thickness 0.15)))
     )
-    (fp_text value Raspberry_PI (at 0 -3.1 90) (layer F.Fab)
+    (fp_text value Raspberry_PI (at 0 -3.1 90) (layer F.Fab) hide
       (effects (font (size 1 1) (thickness 0.15)))
     )
@@
       (effects (font (size 1 1) (thickness 0.15)))
     )
-    (fp_text value I2C_SENS_1 (at 0 -3.1 270) (layer F.Fab)
+    (fp_text value I2C_SENS_1 (at 0 -3.1 270) (layer F.Fab) hide
       (effects (font (size 1 1) (thickness 0.15)))
     )
@@
       (effects (font (size 1 1) (thickness 0.15)))
     )
-    (fp_text value I2C_SENS_1 (at 0 -3.1 270) (layer F.Fab)
+    (fp_text value I2C_SENS_1 (at 0 -3.1 270) (layer F.Fab) hide
       (effects (font (size 1 1) (thickness 0.15)))
     )
@@
       (effects (font (size 1 1) (thickness 0.15)))
     )
-    (fp_text value I2C_SENS_1 (at 0 -3.1 270) (layer F.Fab)
+    (fp_text value I2C_SENS_1 (at 0 -3.1 270) (layer F.Fab) hide
       (effects (font (size 1 1) (thickness 0.15)))
     )
@@
       (effects (font (size 1 1) (thickness 0.15)))
     )
-    (fp_text value CAT24C32WI-GT3 (at 0 -3.72) (layer F.Fab)
+    (fp_text value CAT24C32WI-GT3 (at 0 -3.72) (layer F.Fab) hide
       (effects (font (size 1 1) (thickness 0.15)))
     )
@@
       (effects (font (size 1 1) (thickness 0.15)))
     )
-    (fp_text value CONN_01X04 (at 0 -3.1 90) (layer F.Fab)
+    (fp_text value CONN_01X04 (at 0 -3.1 90) (layer F.Fab) hide
       (effects (font (size 1 1) (thickness 0.15)))
     )
@@
       (effects (font (size 1 1) (thickness 0.15)))
     )
-    (fp_text value TSOP34838 (at 0 -0.5) (layer F.Fab)
+    (fp_text value TSOP34838 (at 0 -0.5) (layer F.Fab) hide
       (effects (font (size 1 1) (thickness 0.15)))
     )
@@
       (effects (font (size 1 1) (thickness 0.15)))
     )
-    (fp_text value MountingHole_2.7mm_M2.5_DIN965_Pad (at 0 3.35) (layer F.Fab)
+    (fp_text value MountingHole_2.7mm_M2.5_DIN965_Pad (at 0 3.35) (layer F.Fab) hide
       (effects (font (size 1 1) (thickness 0.15)))
     )
@@
       (effects (font (size 1 1) (thickness 0.15)))
     )
-    (fp_text value MountingHole_2.7mm_M2.5_DIN965_Pad (at 0 3.35) (layer F.Fab)
+    (fp_text value MountingHole_2.7mm_M2.5_DIN965_Pad (at 0 3.35) (layer F.Fab) hide
       (effects (font (size 1 1) (thickness 0.15)))
     )
@@
       (effects (font (size 1 1) (thickness 0.15)))
     )
-    (fp_text value MountingHole_2.7mm_M2.5_DIN965_Pad (at 0 3.35) (layer F.Fab)
+    (fp_text value MountingHole_2.7mm_M2.5_DIN965_Pad (at 0 3.35) (layer F.Fab) hide
       (effects (font (size 1 1) (thickness 0.15)))
     )
@@
       (effects (font (size 1 1) (thickness 0.15)))
     )
-    (fp_text value MountingHole_2.7mm_M2.5_DIN965_Pad (at 0 3.35) (layer F.Fab)
+    (fp_text value MountingHole_2.7mm_M2.5_DIN965_Pad (at 0 3.35) (layer F.Fab) hide
       (effects (font (size 1 1) (thickness 0.15)))
     )
@@
       (xy -1.693333 -1.524) (xy -1.693333 -1.778) (xy 1.693334 -1.778) (xy 1.693334 1.693334)) (layer F.SilkS) (width 0.01))
   )
+  (gr_text BC817 (at 159.6 86.6) (layer F.Fab)
+    (effects (font (size 0.6 0.6) (thickness 0.125)))
+  )
+  (gr_text 10K (at 159.7 91.6) (layer F.Fab)
+    (effects (font (size 1 1) (thickness 0.25)))
+  )
+  (gr_text 470 (at 169.4 91.7 90) (layer F.Fab)
+    (effects (font (size 1 1) (thickness 0.25)))
+  )
+  (gr_text 4,7pF (at 167.9 96.7) (layer F.Fab)
+    (effects (font (size 1 1) (thickness 0.25)))
+  )
+  (gr_text 100nF (at 210 83.9 90) (layer F.Fab)
+    (effects (font (size 1 0.8) (thickness 0.2)))
+  )
+  (gr_text 1K (at 210 88.9 90) (layer F.Fab)
+    (effects (font (size 1 1) (thickness 0.25)))
+  )
+  (gr_text 4,7K (at 174.5 96.8 90) (layer F.Fab)
+    (effects (font (size 1 1) (thickness 0.25)))
+  )
+  (gr_text 4,7K (at 174.4 91.7 90) (layer F.Fab)
+    (effects (font (size 1 1) (thickness 0.25)))
+  )
+  (gr_text 4,7K (at 203.9 87.9) (layer F.Fab)
+    (effects (font (size 1 1) (thickness 0.25)))
+  )
+  (gr_text 4,7K (at 203.9 83.9) (layer F.Fab)
+    (effects (font (size 1 1) (thickness 0.25)))
+  )
   (gr_text "Rev 1.0 (c) 2017" (at 182.8 102) (layer F.SilkS)
